Commit message: gazebo_launch

File: urdf/fivedofarmzup.xacro (robot description, xacro)
@@ -4,4 +4,5 @@
   <xacro:include filename="$(find fivedofarmzup_description)/urdf/materials.xacro" />
   <xacro:include filename="$(find fivedofarmzup_description)/urdf/fivedofarmzup.trans" />
+  <xacro:include filename="$(find fivedofarmzup_description)/urdf/fivedofarmzup_gazebo.xacro" />
   <link name="base_link">
     <inertial>
@@ -24,7 +25,14 @@
     </collision>
   </link>
-  <gazebo reference="base_link">
-        <material>Gazebo/Blue</material>
-    </gazebo>
+  <!-- <gazebo reference="base_link">
+    <material>Gazebo/Blue</material>
+    <mu1>0.2</mu1>
+    <mu2>0.2</mu2>
+    <self_collide>true</self_collide>
+    <gravity>true</gravity>
+  </gazebo> -->
+  <!-- <gazebo reference="base_link">
+    <material>Gazebo/Blue</material>
+  </gazebo> -->
   <link name="Servo_Bracket_-_U_Shaped_Defaut_v1_1">
     <inertial>
@@ -47,4 +55,11 @@
     </collision>
   </link>
+  <!-- <gazebo reference="Servo_Bracket_-_U_Shaped_Defaut_v1_1">
+    <material>Gazebo/Blue</material>
+    <mu1>0.2</mu1>
+    <mu2>0.2</mu2>
+    <self_collide>true</self_collide>
+    <gravity>true</gravity>
+  </gazebo> -->
   <link name="Standard_Servo__1501MG__v2_1">
     <inertial>
@@ -67,4 +82,11 @@
     </collision>
   </link>
+  <!-- <gazebo reference="Standard_Servo__1501MG__v2_1">
+    <material>Gazebo/Blue</material>
+    <mu1>0.2</mu1>
+    <mu2>0.2</mu2>
+    <self_collide>true</self_collide>
+    <gravity>true</gravity>
+  </gazebo> -->
   <link name="Servo_Bracket_-_U_Shaped_Defaut_v1_2">
     <inertial>
@@ -87,4 +109,11 @@
     </collision>
   </link>
+  <!-- <gazebo reference="Servo_Bracket_-_U_Shaped_Defaut_v1_2">
+    <material>Gazebo/Blue</material>
+    <mu1>0.2</mu1>
+    <mu2>0.2</mu2>
+    <self_collide>true</self_collide>
+    <gravity>true</gravity>
+  </gazebo> -->
   <link name="Standard_Servo__1501MG__v2_2">
     <inertial>
@@ -107,4 +136,11 @@
     </collision>
   </link>
+  <!-- <gazebo reference="Standard_Servo__1501MG__v2_2">
+    <material>Gazebo/Blue</material>
+    <mu1>0.2</mu1>
+    <mu2>0.2</mu2>
+    <self_collide>true</self_collide>
+    <gravity>true</gravity>
+  </gazebo> -->
   <link name="Servo_Bracket_-_U_Shaped_bis_Defaut_v1_1">
     <inertial>
@@ -127,4 +163,11 @@
     </collision>
   </link>
+  <!-- <gazebo reference="Servo_Bracket_-_U_Shaped_bis_Defaut_v1_1">
+    <material>Gazebo/Blue</material>
+    <mu1>0.2</mu1>
+    <mu2>0.2</mu2>
+    <self_collide>true</self_collide>
+    <gravity>true</gravity>
+  </gazebo> -->
   <link name="U_Bracket_Defaut_v1_1">
     <inertial>
@@ -147,4 +190,11 @@
     </collision>
   </link>
+  <!-- <gazebo reference="U_Bracket_Defaut_v1_1">
+    <material>Gazebo/Blue</material>
+    <mu1>0.2</mu1>
+    <mu2>0.2</mu2>
+    <self_collide>true</self_collide>
+    <gravity>true</gravity>
+  </gazebo> -->
   <link name="Standard_Servo__1501MG__v2_3">
     <inertial>
@@ -167,4 +217,11 @@
     </collision>
   </link>
+  <!-- <gazebo reference="Standard_Servo__1501MG__v2_3">
+    <material>Gazebo/Blue</material>
+    <mu1>0.2</mu1>
+    <mu2>0.2</mu2>
+    <self_collide>true</self_collide>
+    <gravity>true</gravity>
+  </gazebo> -->
   <link name="Servo_Bracket_-_Corner_Mount_Defaut_v1_1">
     <inertial>
@@ -187,4 +244,11 @@
     </collision>
   </link>
+  <!-- <gazebo reference="Servo_Bracket_-_Corner_Mount_Defaut_v1_1">
+    <material>Gazebo/Blue</material>
+    <mu1>0.2</mu1>
+    <mu2>0.2</mu2>
+    <self_collide>true</self_collide>
+    <gravity>true</gravity>
+  </gazebo> -->
   <link name="U_Bracket_Defaut_v1_2">
     <inertial>
@@ -207,4 +271,11 @@
     </collision>
   </link>
+  <!-- <gazebo reference="U_Bracket_Defaut_v1_2">
+    <material>Gazebo/Blue</material>
+    <mu1>0.2</mu1>
+    <mu2>0.2</mu2>
+    <self_collide>true</self_collide>
+    <gravity>true</gravity>
+  </gazebo> -->
   <link name="Standard_Servo__1501MG__v2_4">
     <inertial>
@@ -227,4 +298,11 @@
     </collision>
   </link>
+  <!-- <gazebo reference="Standard_Servo__1501MG__v2_4">
+    <material>Gazebo/Blue</material>
+    <mu1>0.2</mu1>
+    <mu2>0.2</mu2>
+    <self_collide>true</self_collide>
+    <gravity>true</gravity>
+  </gazebo> -->
   <link name="Servo_Bracket_-_Corner_Mount_Defaut_v1_2">
     <inertial>
@@ -247,4 +325,11 @@
     </collision>
   </link>
+  <!-- <gazebo reference="Servo_Bracket_-_Corner_Mount_Defaut_v1_2">
+    <material>Gazebo/Blue</material>
+    <mu1>0.2</mu1>
+    <mu2>0.2</mu2>
+    <self_collide>true</self_collide>
+    <gravity>true</gravity>
+  </gazebo> -->
   <link name="Servo_Bracket_-_U_Shaped_Defaut_v1_5">
     <inertial>
@@ -267,4 +352,11 @@
     </collision>
   </link>
+  <!-- <gazebo reference="Servo_Bracket_-_U_Shaped_Defaut_v1_5">
+    <material>Gazebo/Blue</material>
+    <mu1>0.2</mu1>
+    <mu2>0.2</mu2>
+    <self_collide>true</self_collide>
+    <gravity>true</gravity>
+  </gazebo> -->
   <link name="Standard_Servo__1501MG__v2_5">
     <inertial>
@@ -287,4 +379,11 @@
     </collision>
   </link>
+  <!-- <gazebo reference="Standard_Servo__1501MG__v2_5">
+    <material>Gazebo/Blue</material>
+    <mu1>0.2</mu1>
+    <mu2>0.2</mu2>
+    <self_collide>true</self_collide>
+    <gravity>true</gravity>
+  </gazebo> -->
   <link name="Servo_Bracket_-_U_Shaped_Defaut_v1_3">
     <inertial>
@@ -307,4 +406,11 @@
     </collision>
   </link>
+  <!-- <gazebo reference="Servo_Bracket_-_U_Shaped_Defaut_v1_3">
+    <material>Gazebo/Blue</material>
+    <mu1>0.2</mu1>
+    <mu2>0.2</mu2>
+    <self_collide>true</self_collide>
+    <gravity>true</gravity>
+  </gazebo> -->
   <link name="Servo_Bracket_-_U_Shaped_Defaut_v1_4">
     <inertial>
@@ -327,4 +433,11 @@
     </collision>
   </link>
+  <!-- <gazebo reference="Servo_Bracket_-_U_Shaped_Defaut_v1_4">
+    <material>Gazebo/Blue</material>
+    <mu1>0.2</mu1>
+    <mu2>0.2</mu2>
+    <self_collide>true</self_collide>
+    <gravity>true</gravity>
+  </gazebo> -->
   <link name="Gripz_v2_1">
     <inertial>
@@ -347,4 +460,11 @@
     </collision>
   </link>
+  <!-- <gazebo reference="Gripz_v2_1">
+    <material>Gazebo/Blue</material>
+    <mu1>0.2</mu1>
+    <mu2>0.2</mu2>
+    <self_collide>true</self_collide>
+    <gravity>true</gravity>
+  </gazebo> -->
   <link name="left-gripper_v3_1">
     <inertial>
@@ -367,4 +487,11 @@
     </collision>
   </link>
+  <!-- <gazebo reference="left-gripper_v3_1">
+    <material>Gazebo/Blue</material>
+    <mu1>0.2</mu1>
+    <mu2>0.2</mu2>
+    <self_collide>true</self_collide>
+    <gravity>true</gravity>
+  </gazebo> -->
   <link name="right-gripper_v2_1">
     <inertial>
@@ -387,4 +514,11 @@
     </collision>
   </link>
+  <!-- <gazebo reference="right-gripper_v2_1">
+    <material>Gazebo/Blue</material>
+    <mu1>0.2</mu1>
+    <mu2>0.2</mu2>
+    <self_collide>true</self_collide>
+    <gravity>true</gravity>
+  </gazebo> -->
   <joint name="Rigid 1" type="fixed">
     <origin xyz="0.008257 -0.025556 0.025987" rpy="0 0 0"/>
@@ -469,5 +603,5 @@
     <child link="Servo_Bracket_-_U_Shaped_Defaut_v1_4"/>
   </joint>
-    <joint name="Revolute 19" type="revolute">
+  <joint name="Revolute 19" type="revolute">
     <origin xyz="0.006804 -0.015812 0.015774" rpy="0 0 0"/>
     <parent link="Standard_Servo__1501MG__v2_5"/>
@@ -481,4 +615,5 @@
     <child link="left-gripper_v3_1"/>
     <axis xyz="0.574019 0.789827 0.216045"/>
+    <limit upper="1.0" lower="-1.0" effort="100" velocity="100"/>
   </joint>
   <joint name="Revolute 22" type="continuous">
@@ -486,4 +621,5 @@
     <parent link="Gripz_v2_1"/>
     <child link="right-gripper_v2_1"/>
+    <mimic joint = "Revolute 21" multiplier = "-1" />
     <axis xyz="0.574019 0.789827 0.216045"/>
   </joint>

Commit message: gazebo launch

File: urdf/fivedofarmzup.xacro (robot description, xacro)
@@ -25,14 +25,4 @@
     </collision>
   </link>
-  <!-- <gazebo reference="base_link">
-    <material>Gazebo/Blue</material>
-    <mu1>0.2</mu1>
-    <mu2>0.2</mu2>
-    <self_collide>true</self_collide>
-    <gravity>true</gravity>
-  </gazebo> -->
-  <!-- <gazebo reference="base_link">
-    <material>Gazebo/Blue</material>
-  </gazebo> -->
   <link name="Servo_Bracket_-_U_Shaped_Defaut_v1_1">
     <inertial>
@@ -55,11 +45,4 @@
     </collision>
   </link>
-  <!-- <gazebo reference="Servo_Bracket_-_U_Shaped_Defaut_v1_1">
-    <material>Gazebo/Blue</material>
-    <mu1>0.2</mu1>
-    <mu2>0.2</mu2>
-    <self_collide>true</self_collide>
-    <gravity>true</gravity>
-  </gazebo> -->
   <link name="Standard_Servo__1501MG__v2_1">
     <inertial>
@@ -82,11 +65,4 @@
     </collision>
   </link>
-  <!-- <gazebo reference="Standard_Servo__1501MG__v2_1">
-    <material>Gazebo/Blue</material>
-    <mu1>0.2</mu1>
-    <mu2>0.2</mu2>
-    <self_collide>true</self_collide>
-    <gravity>true</gravity>
-  </gazebo> -->
   <link name="Servo_Bracket_-_U_Shaped_Defaut_v1_2">
     <inertial>
@@ -109,11 +85,4 @@
     </collision>
   </link>
-  <!-- <gazebo reference="Servo_Bracket_-_U_Shaped_Defaut_v1_2">
-    <material>Gazebo/Blue</material>
-    <mu1>0.2</mu1>
-    <mu2>0.2</mu2>
-    <self_collide>true</self_collide>
-    <gravity>true</gravity>
-  </gazebo> -->
   <link name="Standard_Servo__1501MG__v2_2">
     <inertial>
@@ -136,11 +105,4 @@
     </collision>
   </link>
-  <!-- <gazebo reference="Standard_Servo__1501MG__v2_2">
-    <material>Gazebo/Blue</material>
-    <mu1>0.2</mu1>
-    <mu2>0.2</mu2>
-    <self_collide>true</self_collide>
-    <gravity>true</gravity>
-  </gazebo> -->
   <link name="Servo_Bracket_-_U_Shaped_bis_Defaut_v1_1">
     <inertial>
@@ -163,11 +125,4 @@
     </collision>
   </link>
-  <!-- <gazebo reference="Servo_Bracket_-_U_Shaped_bis_Defaut_v1_1">
-    <material>Gazebo/Blue</material>
-    <mu1>0.2</mu1>
-    <mu2>0.2</mu2>
-    <self_collide>true</self_collide>
-    <gravity>true</gravity>
-  </gazebo> -->
   <link name="U_Bracket_Defaut_v1_1">
     <inertial>
@@ -190,11 +145,4 @@
     </collision>
   </link>
-  <!-- <gazebo reference="U_Bracket_Defaut_v1_1">
-    <material>Gazebo/Blue</material>
-    <mu1>0.2</mu1>
-    <mu2>0.2</mu2>
-    <self_collide>true</self_collide>
-    <gravity>true</gravity>
-  </gazebo> -->
   <link name="Standard_Servo__1501MG__v2_3">
     <inertial>
@@ -217,11 +165,4 @@
     </collision>
   </link>
-  <!-- <gazebo reference="Standard_Servo__1501MG__v2_3">
-    <material>Gazebo/Blue</material>
-    <mu1>0.2</mu1>
-    <mu2>0.2</mu2>
-    <self_collide>true</self_collide>
-    <gravity>true</gravity>
-  </gazebo> -->
   <link name="Servo_Bracket_-_Corner_Mount_Defaut_v1_1">
     <inertial>
@@ -244,11 +185,4 @@
     </collision>
   </link>
-  <!-- <gazebo reference="Servo_Bracket_-_Corner_Mount_Defaut_v1_1">
-    <material>Gazebo/Blue</material>
-    <mu1>0.2</mu1>
-    <mu2>0.2</mu2>
-    <self_collide>true</self_collide>
-    <gravity>true</gravity>
-  </gazebo> -->
   <link name="U_Bracket_Defaut_v1_2">
     <inertial>
@@ -271,11 +205,4 @@
     </collision>
   </link>
-  <!-- <gazebo reference="U_Bracket_Defaut_v1_2">
-    <material>Gazebo/Blue</material>
-    <mu1>0.2</mu1>
-    <mu2>0.2</mu2>
-    <self_collide>true</self_collide>
-    <gravity>true</gravity>
-  </gazebo> -->
   <link name="Standard_Servo__1501MG__v2_4">
     <inertial>
@@ -298,11 +225,4 @@
     </collision>
   </link>
-  <!-- <gazebo reference="Standard_Servo__1501MG__v2_4">
-    <material>Gazebo/Blue</material>
-    <mu1>0.2</mu1>
-    <mu2>0.2</mu2>
-    <self_collide>true</self_collide>
-    <gravity>true</gravity>
-  </gazebo> -->
   <link name="Servo_Bracket_-_Corner_Mount_Defaut_v1_2">
     <inertial>
@@ -325,11 +245,4 @@
     </collision>
   </link>
-  <!-- <gazebo reference="Servo_Bracket_-_Corner_Mount_Defaut_v1_2">
-    <material>Gazebo/Blue</material>
-    <mu1>0.2</mu1>
-    <mu2>0.2</mu2>
-    <self_collide>true</self_collide>
-    <gravity>true</gravity>
-  </gazebo> -->
   <link name="Servo_Bracket_-_U_Shaped_Defaut_v1_5">
     <inertial>
@@ -352,11 +265,4 @@
     </collision>
   </link>
-  <!-- <gazebo reference="Servo_Bracket_-_U_Shaped_Defaut_v1_5">
-    <material>Gazebo/Blue</material>
-    <mu1>0.2</mu1>
-    <mu2>0.2</mu2>
-    <self_collide>true</self_collide>
-    <gravity>true</gravity>
-  </gazebo> -->
   <link name="Standard_Servo__1501MG__v2_5">
     <inertial>
@@ -379,11 +285,4 @@
     </collision>
   </link>
-  <!-- <gazebo reference="Standard_Servo__1501MG__v2_5">
-    <material>Gazebo/Blue</material>
-    <mu1>0.2</mu1>
-    <mu2>0.2</mu2>
-    <self_collide>true</self_collide>
-    <gravity>true</gravity>
-  </gazebo> -->
   <link name="Servo_Bracket_-_U_Shaped_Defaut_v1_3">
     <inertial>
@@ -406,11 +305,4 @@
     </collision>
   </link>
-  <!-- <gazebo reference="Servo_Bracket_-_U_Shaped_Defaut_v1_3">
-    <material>Gazebo/Blue</material>
-    <mu1>0.2</mu1>
-    <mu2>0.2</mu2>
-    <self_collide>true</self_collide>
-    <gravity>true</gravity>
-  </gazebo> -->
   <link name="Servo_Bracket_-_U_Shaped_Defaut_v1_4">
     <inertial>
@@ -433,11 +325,4 @@
     </collision>
   </link>
-  <!-- <gazebo reference="Servo_Bracket_-_U_Shaped_Defaut_v1_4">
-    <material>Gazebo/Blue</material>
-    <mu1>0.2</mu1>
-    <mu2>0.2</mu2>
-    <self_collide>true</self_collide>
-    <gravity>true</gravity>
-  </gazebo> -->
   <link name="Gripz_v2_1">
     <inertial>
@@ -460,11 +345,4 @@
     </collision>
   </link>
-  <!-- <gazebo reference="Gripz_v2_1">
-    <material>Gazebo/Blue</material>
-    <mu1>0.2</mu1>
-    <mu2>0.2</mu2>
-    <self_collide>true</self_collide>
-    <gravity>true</gravity>
-  </gazebo> -->
   <link name="left-gripper_v3_1">
     <inertial>
@@ -487,11 +365,4 @@
     </collision>
   </link>
-  <!-- <gazebo reference="left-gripper_v3_1">
-    <material>Gazebo/Blue</material>
-    <mu1>0.2</mu1>
-    <mu2>0.2</mu2>
-    <self_collide>true</self_collide>
-    <gravity>true</gravity>
-  </gazebo> -->
   <link name="right-gripper_v2_1">
     <inertial>
@@ -514,11 +385,4 @@
     </collision>
   </link>
-  <!-- <gazebo reference="right-gripper_v2_1">
-    <material>Gazebo/Blue</material>
-    <mu1>0.2</mu1>
-    <mu2>0.2</mu2>
-    <self_collide>true</self_collide>
-    <gravity>true</gravity>
-  </gazebo> -->
   <joint name="Rigid 1" type="fixed">
     <origin xyz="0.008257 -0.025556 0.025987" rpy="0 0 0"/>

File: urdf/fivedofarmzup_gazebo.xacro (robot description, xacro)
@@ -12,5 +12,5 @@
     <xacro:property name="camera_color" value="Gazebo/Silver" />
     <gazebo reference="base_link">
-        <material>Gazebo/Blue</material>
+        <material>Gazebo/Green</material>
         <mu1>0.2</mu1>
         <mu2>0.2</mu2>
@@ -19,5 +19,5 @@
     </gazebo>
     <gazebo reference="Servo_Bracket_-_U_Shaped_Defaut_v1_1">
-        <material>Gazebo/Blue</material>
+        <material>Gazebo/Red</material>
         <mu1>0.2</mu1>
         <mu2>0.2</mu2>
@@ -26,5 +26,5 @@
     </gazebo>
     <gazebo reference="Standard_Servo__1501MG__v2_1">
-        <material>Gazebo/Blue</material>
+        <material>Gazebo/Black</material>
         <mu1>0.2</mu1>
         <mu2>0.2</mu2>
@@ -33,5 +33,5 @@
     </gazebo>
     <gazebo reference="Servo_Bracket_-_U_Shaped_Defaut_v1_2">
-        <material>Gazebo/Blue</material>
+        <material>Gazebo/Red</material>
         <mu1>0.2</mu1>
         <mu2>0.2</mu2>
@@ -40,5 +40,5 @@
     </gazebo>
     <gazebo reference="Standard_Servo__1501MG__v2_2">
-        <material>Gazebo/Blue</material>
+        <material>Gazebo/Black</material>
         <mu1>0.2</mu1>
         <mu2>0.2</mu2>
